Commit message: controller commit

File: cartpole_urdf/urdf/cartpole.urdf (robot description, URDF)
Before this commit: robot cart_pole, 3 links, 2 joints
Links:
- added link dummy_link, mass 0.0001; collision box size=0.001 0.001 0.001; visual box size=0.001 0.001 0.001
- link cart_link: mass 1 -> 10
- link pole_link: mass 0.1 -> 2
Joints:
- added joint dummy_joint: type fixed, parent base_link, child dummy_link, origin xyz=0 0 0.05
- joint cart_joint: axis (none) -> 1 0 0; limit (none) -> lower=-5 upper=5 effort=10 velocity=1; type fixed -> prismatic

Commit message: LQR control

File: cartpole_urdf/urdf/cartpole.urdf (robot description, URDF)
Before this commit: robot cart_pole, 4 links, 3 joints
Links:
- removed link base_link
- added link world
- link dummy_link: mass 0.0001 -> 0.1; geometry visual box size=1 0.1 0.01
Joints:
- joint cart_joint: limit lower=-5 upper=5 effort=10 velocity=1 -> lower=-10 upper=10 effort=600 velocity=200; parent base_link -> world
- joint dummy_joint: parent base_link -> world
- joint pole_joint: origin xyz=0 0 0.05 rpy=0 0 0 -> xyz=0 0 0.05 rpy=0 0.25 0

Commit message: stl & qp solver

File: cartpole_urdf/urdf/cartpole.urdf (robot description, URDF)
Before this commit: robot cart_pole, 4 links, 3 joints
Links:
- added link ruler, mass 1; visual mesh filename=/home/obot/catkin_ws/src/cartpole_urdf/meshes/CP_ruler_cut.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 scale=0.001 0.001 0.001
- link dummy_link: geometry visual box size=20 0.01 0.05
Joints:
- added joint ruler_joint: type fixed, parent world, child ruler, origin xyz=-10 1 0.0 rpy=1.57079632679 0 0
- joint dummy_joint: origin xyz=0 0 0.05 -> xyz=0 0 0.025

Commit message: QP controller

File: cartpole_urdf/urdf/cartpole.urdf (robot description, URDF)
Before this commit: robot cart_pole, 5 links, 4 joints
Links:
- link pole_link: mass 2 -> 1
